File: PCB/PhobGCC.kicad_sch (KiCad schematic)
At the start: 46 parts, among them J1 Conn_01x06_Female, J2 Conn_01x04_Female, J3 Conn_01x01_Male, J4 Conn_01x01_Male, J6 10118194-0001LF, SW1 A, SW10 Dup, SW11 Dright, SW12 Ddown, SW2 B, SW3 X, SW4 Y, SW5 Start, SW6 L, SW7 R, SW8 1825027-5, SW9 Dleft, U1 Teensy3.2, U2 2x DRV5053CAQLPGM Hall Effect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, U3 2.5V LDO

Commit message: cleaned manufacturing files for the v1.1 board
Parts:
- C1, C2, C3, C4, C5, C6, C7: value 2200p -> 0.047u
- R1, R2: value 10k -> 2k
- U3: value 2.5V LDO -> ME6206A25XG
Changed lines of the file:
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@@
       (effects (font (size 1.27 1.27)) (justify left))
     )
-    (property "Value" "2200p" (id 1) (at 43.561 177.673 0)
+    (property "Value" "0.047u" (id 1) (at 43.561 177.673 0)
       (effects (font (size 1.27 1.27)) (justify left))
     )
@@
       (effects (font (size 1.27 1.27)) (justify left))
     )
-    (property "Value" "2200p" (id 1) (at 63.881 177.673 0)
+    (property "Value" "0.047u" (id 1) (at 63.881 177.673 0)
       (effects (font (size 1.27 1.27)) (justify left))
     )
@@
       (effects (font (size 1.27 1.27)) (justify left))
     )
-    (property "Value" "2200p" (id 1) (at 71.501 177.673 0)
+    (property "Value" "0.047u" (id 1) (at 71.501 177.673 0)
       (effects (font (size 1.27 1.27)) (justify left))
     )
@@
       (effects (font (size 1.27 1.27)) (justify left))
     )
-    (property "Value" "2200p" (id 1) (at 79.121 177.673 0)
+    (property "Value" "0.047u" (id 1) (at 79.121 177.673 0)
       (effects (font (size 1.27 1.27)) (justify left))
     )
@@
       (effects (font (size 1.27 1.27)) (justify left))
     )
-    (property "Value" "2200p" (id 1) (at 86.741 177.673 0)
+    (property "Value" "0.047u" (id 1) (at 86.741 177.673 0)
       (effects (font (size 1.27 1.27)) (justify left))
     )
@@
       (effects (font (size 1.27 1.27)) (justify left))
     )
-    (property "Value" "2200p" (id 1) (at 101.981 177.673 0)
+    (property "Value" "0.047u" (id 1) (at 101.981 177.673 0)
       (effects (font (size 1.27 1.27)) (justify left))
     )
@@
     (in_bom yes) (on_board yes)
     (property "Reference" "U3" (id 0) (at 83.82 22.4282 0))
-    (property "Value" "2.5V LDO" (id 1) (at 83.82 24.7396 0))
+    (property "Value" "ME6206A25XG" (id 1) (at 83.82 24.7396 0))
     (property "Footprint" "Package_TO_SOT_SMD:SOT-23_Handsoldering" (id 2) (at 83.82 31.75 0)
       (effects (font (size 1.27 1.27)) hide)
@@
     (in_bom yes) (on_board yes)
     (property "Reference" "R1" (id 0) (at 36.83 163.6522 90))
-    (property "Value" "10k" (id 1) (at 36.83 165.9636 90))
+    (property "Value" "2k" (id 1) (at 36.83 165.9636 90))
     (property "Footprint" "Resistor_SMD:R_0603_1608Metric" (id 2) (at 36.83 167.132 90)
       (effects (font (size 1.27 1.27)) hide)
@@
     (in_bom yes) (on_board yes)
     (property "Reference" "R2" (id 0) (at 55.88 163.6522 90))
-    (property "Value" "10k" (id 1) (at 55.88 165.9636 90))
+    (property "Value" "2k" (id 1) (at 55.88 165.9636 90))
     (property "Footprint" "Resistor_SMD:R_0603_1608Metric" (id 2) (at 55.88 167.132 90)
       (effects (font (size 1.27 1.27)) hide)
@@
       (effects (font (size 1.27 1.27)) (justify left))
     )
-    (property "Value" "2200p" (id 1) (at 63.881 41.783 0)
+    (property "Value" "0.047u" (id 1) (at 63.881 41.783 0)
       (effects (font (size 1.27 1.27)) (justify left))
     )
@@
     )
     (path "/00000000-0000-0000-0000-000061652d1a"
-      (reference "C1") (unit 1) (value "2200p") (footprint "Capacitors_SMD:C_0603_HandSoldering")
+      (reference "C1") (unit 1) (value "0.047u") (footprint "Capacitors_SMD:C_0603_HandSoldering")
     )
     (path "/00000000-0000-0000-0000-00006165460d"
-      (reference "C2") (unit 1) (value "2200p") (footprint "Capacitors_SMD:C_0603_HandSoldering")
+      (reference "C2") (unit 1) (value "0.047u") (footprint "Capacitors_SMD:C_0603_HandSoldering")
     )
     (path "/00000000-0000-0000-0000-0000616548ab"
-      (reference "C3") (unit 1) (value "2200p") (footprint "Capacitors_SMD:C_0603_HandSoldering")
+      (reference "C3") (unit 1) (value "0.047u") (footprint "Capacitors_SMD:C_0603_HandSoldering")
     )
     (path "/00000000-0000-0000-0000-000061654b98"
-      (reference "C4") (unit 1) (value "2200p") (footprint "Capacitors_SMD:C_0603_HandSoldering")
+      (reference "C4") (unit 1) (value "0.047u") (footprint "Capacitors_SMD:C_0603_HandSoldering")
     )
     (path "/00000000-0000-0000-0000-000061654de5"
-      (reference "C5") (unit 1) (value "2200p") (footprint "Capacitors_SMD:C_0603_HandSoldering")
+      (reference "C5") (unit 1) (value "0.047u") (footprint "Capacitors_SMD:C_0603_HandSoldering")
     )
     (path "/00000000-0000-0000-0000-000061f792e8"
-      (reference "C6") (unit 1) (value "2200p") (footprint "Capacitors_SMD:C_0603_HandSoldering")
+      (reference "C6") (unit 1) (value "0.047u") (footprint "Capacitors_SMD:C_0603_HandSoldering")
     )
     (path "/00000000-0000-0000-0000-000061655620"
-      (reference "C7") (unit 1) (value "2200p") (footprint "Capacitors_SMD:C_0603_HandSoldering")
+      (reference "C7") (unit 1) (value "0.047u") (footprint "Capacitors_SMD:C_0603_HandSoldering")
     )
     (path "/00000000-0000-0000-0000-000061ed6d60"
@@
     )
     (path "/00000000-0000-0000-0000-000061f268c6"
-      (reference "R1") (unit 1) (value "10k") (footprint "Resistor_SMD:R_0603_1608Metric")
+      (reference "R1") (unit 1) (value "2k") (footprint "Resistor_SMD:R_0603_1608Metric")
     )
     (path "/00000000-0000-0000-0000-000061f3dce6"
-      (reference "R2") (unit 1) (value "10k") (footprint "Resistor_SMD:R_0603_1608Metric")
+      (reference "R2") (unit 1) (value "2k") (footprint "Resistor_SMD:R_0603_1608Metric")
     )
     (path "/00000000-0000-0000-0000-000061575265"
@@
     )
     (path "/00000000-0000-0000-0000-000061e87b70"
-      (reference "U3") (unit 1) (value "2.5V LDO") (footprint "Package_TO_SOT_SMD:SOT-23_Handsoldering")
-    )
-  )
+      (reference "U3") (unit 1) (value "ME6206A25XG") (footprint "Package_TO_SOT_SMD:SOT-23_Handsoldering")
+    )
+  )
